File: Keyboard_v1/_autosave-Keyboard_v1.kicad_pcb (KiCad board)
At the start: 2 copper layers, 174 parts, among them SW1 SW_Push, U1 ATmega32U4-A, Y1 16MHz

Commit message: all rows and cols connected to MCU
Parts:
- moved R1 39.3 mm to (418.4, 167.4), turned to 180 degrees
- moved C3 28.8 mm to (422.1, 189.3)
- moved C2 21.9 mm to (422.1, 193.3)
- moved C6 21.8 mm to (414.3, 192.1), turned to 90 degrees
- moved R2 19.4 mm to (401.6, 163.5)
- moved U1 18.9 mm to (414.3, 177.9), turned to 0 degrees
- moved Y1 15.7 mm to (410.4, 192.1), turned to 180 degrees
- moved R3 15.3 mm to (404.8, 163.5)
- moved SW1 9.79 mm to (394.5, 169.1)
- moved D5 9.42 mm to (141.7, 237.4)
- moved C7 9.35 mm to (405.6, 192.1), turned to -90 degrees
- moved F1 9.35 mm to (410.3, 166.1)
- moved C1 8.85 mm to (402.4, 179.4), turned to 90 degrees
- moved C4 8.28 mm to (422.1, 201.2), turned to 180 degrees
- moved USB1 8.09 mm to (404.8, 152.6), turned to -90 degrees
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Connections:
- D1 pad 1: /Sheet: Switch Matrix/ROW0 -> ROW0
- D10 pad 1: /Sheet: Switch Matrix/ROW3 -> ROW3
- D11 pad 1: /Sheet: Switch Matrix/ROW4 -> ROW4
- D12 pad 1: /Sheet: Switch Matrix/ROW5 -> ROW5
- D13 pad 1: /Sheet: Switch Matrix/ROW0 -> ROW0
- D14 pad 1: /Sheet: Switch Matrix/ROW1 -> ROW1
- D15 pad 1: /Sheet: Switch Matrix/ROW2 -> ROW2
- D16 pad 1: /Sheet: Switch Matrix/ROW3 -> ROW3
- D17 pad 1: /Sheet: Switch Matrix/ROW4 -> ROW4
- D18 pad 1: /Sheet: Switch Matrix/ROW5 -> ROW5
- D19 pad 1: /Sheet: Switch Matrix/ROW0 -> ROW0
- D2 pad 1: /Sheet: Switch Matrix/ROW1 -> ROW1
- D20 pad 1: /Sheet: Switch Matrix/ROW1 -> ROW1
- D21 pad 1: /Sheet: Switch Matrix/ROW2 -> ROW2
- D22 pad 1: /Sheet: Switch Matrix/ROW3 -> ROW3
- D23 pad 1: /Sheet: Switch Matrix/ROW4 -> ROW4
- D24 pad 1: /Sheet: Switch Matrix/ROW5 -> ROW5
- D25 pad 1: /Sheet: Switch Matrix/ROW0 -> ROW0
- D26 pad 1: /Sheet: Switch Matrix/ROW1 -> ROW1
- D27 pad 1: /Sheet: Switch Matrix/ROW2 -> ROW2
- D28 pad 1: /Sheet: Switch Matrix/ROW3 -> ROW3
- D29 pad 1: /Sheet: Switch Matrix/ROW4 -> ROW4
- D3 pad 1: /Sheet: Switch Matrix/ROW2 -> ROW2
- D30 pad 1: /Sheet: Switch Matrix/ROW5 -> ROW5
- D31 pad 1: /Sheet: Switch Matrix/ROW0 -> ROW0
- D32 pad 1: /Sheet: Switch Matrix/ROW1 -> ROW1
- D33 pad 1: /Sheet: Switch Matrix/ROW2 -> ROW2
- D34 pad 1: /Sheet: Switch Matrix/ROW3 -> ROW3
- D35 pad 1: /Sheet: Switch Matrix/ROW4 -> ROW4
- D36 pad 1: /Sheet: Switch Matrix/ROW5 -> ROW5
- D37 pad 1: /Sheet: Switch Matrix/ROW0 -> ROW0
- D38 pad 1: /Sheet: Switch Matrix/ROW1 -> ROW1
- D39 pad 1: /Sheet: Switch Matrix/ROW2 -> ROW2
- D4 pad 1: /Sheet: Switch Matrix/ROW3 -> ROW3
- D40 pad 1: /Sheet: Switch Matrix/ROW3 -> ROW3
- D41 pad 1: /Sheet: Switch Matrix/ROW4 -> ROW4
- D42 pad 1: /Sheet: Switch Matrix/ROW5 -> ROW5
- D43 pad 1: /Sheet: Switch Matrix/ROW0 -> ROW0
- D44 pad 1: /Sheet: Switch Matrix/ROW1 -> ROW1
- D45 pad 1: /Sheet: Switch Matrix/ROW2 -> ROW2
- D46 pad 1: /Sheet: Switch Matrix/ROW3 -> ROW3
- D47 pad 1: /Sheet: Switch Matrix/ROW4 -> ROW4
- D48 pad 1: /Sheet: Switch Matrix/ROW5 -> ROW5
- D49 pad 1: /Sheet: Switch Matrix/ROW0 -> ROW0
- D5 pad 1: /Sheet: Switch Matrix/ROW4 -> ROW4
- D50 pad 1: /Sheet: Switch Matrix/ROW1 -> ROW1
- D51 pad 1: /Sheet: Switch Matrix/ROW2 -> ROW2
- D52 pad 1: /Sheet: Switch Matrix/ROW3 -> ROW3
- D53 pad 1: /Sheet: Switch Matrix/ROW4 -> ROW4
- D54 pad 1: /Sheet: Switch Matrix/ROW5 -> ROW5
- D55 pad 1: /Sheet: Switch Matrix/ROW0 -> ROW0
- D56 pad 1: /Sheet: Switch Matrix/ROW1 -> ROW1
- D57 pad 1: /Sheet: Switch Matrix/ROW2 -> ROW2
- D58 pad 1: /Sheet: Switch Matrix/ROW3 -> ROW3
- D59 pad 1: /Sheet: Switch Matrix/ROW4 -> ROW4
- D6 pad 1: /Sheet: Switch Matrix/ROW5 -> ROW5
- D60 pad 1: /Sheet: Switch Matrix/ROW5 -> ROW5
- D61 pad 1: /Sheet: Switch Matrix/ROW0 -> ROW0
- D62 pad 1: /Sheet: Switch Matrix/ROW1 -> ROW1
- D63 pad 1: /Sheet: Switch Matrix/ROW2 -> ROW2
- D64 pad 1: /Sheet: Switch Matrix/ROW3 -> ROW3
- D65 pad 1: /Sheet: Switch Matrix/ROW4 -> ROW4
- D66 pad 1: /Sheet: Switch Matrix/ROW5 -> ROW5
- D67 pad 1: /Sheet: Switch Matrix/ROW0 -> ROW0
- D68 pad 1: /Sheet: Switch Matrix/ROW1 -> ROW1
- D69 pad 1: /Sheet: Switch Matrix/ROW2 -> ROW2
- D7 pad 1: /Sheet: Switch Matrix/ROW0 -> ROW0
- D70 pad 1: /Sheet: Switch Matrix/ROW3 -> ROW3
- D71 pad 1: /Sheet: Switch Matrix/ROW4 -> ROW4
- D72 pad 1: /Sheet: Switch Matrix/ROW0 -> ROW0
- D73 pad 1: /Sheet: Switch Matrix/ROW1 -> ROW1
- D74 pad 1: /Sheet: Switch Matrix/ROW2 -> ROW2
- D75 pad 1: /Sheet: Switch Matrix/ROW3 -> ROW3
- D76 pad 1: /Sheet: Switch Matrix/ROW4 -> ROW4
- D77 pad 1: /Sheet: Switch Matrix/ROW0 -> ROW0
- D78 pad 1: /Sheet: Switch Matrix/ROW1 -> ROW1
- D79 pad 1: /Sheet: Switch Matrix/ROW2 -> ROW2
- D8 pad 1: /Sheet: Switch Matrix/ROW1 -> ROW1
- D9 pad 1: /Sheet: Switch Matrix/ROW2 -> ROW2
- MX1 pad 1: /Sheet: Switch Matrix/COL0 -> COL0
- MX10 pad 1: /Sheet: Switch Matrix/COL1 -> COL1
- MX11 pad 1: /Sheet: Switch Matrix/COL1 -> COL1
- MX12 pad 1: /Sheet: Switch Matrix/COL1 -> COL1
- MX13 pad 1: /Sheet: Switch Matrix/COL2 -> COL2
- MX14 pad 1: /Sheet: Switch Matrix/COL2 -> COL2
- MX15 pad 1: /Sheet: Switch Matrix/COL2 -> COL2
- MX16 pad 1: /Sheet: Switch Matrix/COL2 -> COL2
- MX17 pad 1: /Sheet: Switch Matrix/COL2 -> COL2
- MX18 pad 1: /Sheet: Switch Matrix/COL2 -> COL2
- MX19 pad 1: /Sheet: Switch Matrix/COL3 -> COL3
- MX2 pad 1: /Sheet: Switch Matrix/COL0 -> COL0
- MX20 pad 1: /Sheet: Switch Matrix/COL3 -> COL3
- MX21 pad 1: /Sheet: Switch Matrix/COL3 -> COL3
- MX22 pad 1: /Sheet: Switch Matrix/COL3 -> COL3
- MX23 pad 1: /Sheet: Switch Matrix/COL3 -> COL3
- MX24 pad 1: /Sheet: Switch Matrix/COL3 -> COL3
- MX25 pad 1: /Sheet: Switch Matrix/COL4 -> COL4
- MX26 pad 1: /Sheet: Switch Matrix/COL4 -> COL4
- MX27 pad 1: /Sheet: Switch Matrix/COL4 -> COL4
- MX28 pad 1: /Sheet: Switch Matrix/COL4 -> COL4
- MX29 pad 1: /Sheet: Switch Matrix/COL4 -> COL4
- MX3 pad 1: /Sheet: Switch Matrix/COL0 -> COL0
- MX30 pad 1: /Sheet: Switch Matrix/COL4 -> COL4
- MX31 pad 1: /Sheet: Switch Matrix/COL5 -> COL5
- MX32 pad 1: /Sheet: Switch Matrix/COL5 -> COL5
- MX33 pad 1: /Sheet: Switch Matrix/COL5 -> COL5
- MX34 pad 1: /Sheet: Switch Matrix/COL5 -> COL5
- MX35 pad 1: /Sheet: Switch Matrix/COL5 -> COL5
- MX36 pad 1: /Sheet: Switch Matrix/COL5 -> COL5
- MX37 pad 1: /Sheet: Switch Matrix/COL6 -> COL6
- MX38 pad 1: /Sheet: Switch Matrix/COL6 -> COL6
- MX39 pad 1: /Sheet: Switch Matrix/COL6 -> COL6
- MX4 pad 1: /Sheet: Switch Matrix/COL0 -> COL0
- MX40 pad 1: /Sheet: Switch Matrix/COL6 -> COL6
- MX41 pad 1: /Sheet: Switch Matrix/COL6 -> COL6
- MX42 pad 1: /Sheet: Switch Matrix/COL6 -> COL6
- MX43 pad 1: /Sheet: Switch Matrix/COL7 -> COL7
- MX44 pad 1: /Sheet: Switch Matrix/COL7 -> COL7
- MX45 pad 1: /Sheet: Switch Matrix/COL7 -> COL7
- MX46 pad 1: /Sheet: Switch Matrix/COL7 -> COL7
- MX47 pad 1: /Sheet: Switch Matrix/COL7 -> COL7
- MX48 pad 1: /Sheet: Switch Matrix/COL7 -> COL7
- MX49 pad 1: /Sheet: Switch Matrix/COL8 -> COL8
- MX5 pad 1: /Sheet: Switch Matrix/COL0 -> COL0
- MX50 pad 1: /Sheet: Switch Matrix/COL8 -> COL8
- MX51 pad 1: /Sheet: Switch Matrix/COL8 -> COL8
- MX52 pad 1: /Sheet: Switch Matrix/COL8 -> COL8
- MX53 pad 1: /Sheet: Switch Matrix/COL8 -> COL8
- MX54 pad 1: /Sheet: Switch Matrix/COL8 -> COL8
- MX55 pad 1: /Sheet: Switch Matrix/COL9 -> COL9
- MX56 pad 1: /Sheet: Switch Matrix/COL9 -> COL9
- MX57 pad 1: /Sheet: Switch Matrix/COL9 -> COL9
- MX58 pad 1: /Sheet: Switch Matrix/COL9 -> COL9
- MX59 pad 1: /Sheet: Switch Matrix/COL9 -> COL9
- MX6 pad 1: /Sheet: Switch Matrix/COL0 -> COL0
- MX60 pad 1: /Sheet: Switch Matrix/COL9 -> COL9
- MX61 pad 1: /Sheet: Switch Matrix/COL10 -> COL10
- MX62 pad 1: /Sheet: Switch Matrix/COL10 -> COL10
- MX63 pad 1: /Sheet: Switch Matrix/COL10 -> COL10
- MX64 pad 1: /Sheet: Switch Matrix/COL10 -> COL10
- MX65 pad 1: /Sheet: Switch Matrix/COL10 -> COL10
- MX66 pad 1: /Sheet: Switch Matrix/COL10 -> COL10
- MX67 pad 1: /Sheet: Switch Matrix/COL11 -> COL11
- MX68 pad 1: /Sheet: Switch Matrix/COL11 -> COL11
- MX69 pad 1: /Sheet: Switch Matrix/COL11 -> COL11
- MX7 pad 1: /Sheet: Switch Matrix/COL1 -> COL1
- MX70 pad 1: /Sheet: Switch Matrix/COL11 -> COL11
- MX71 pad 1: /Sheet: Switch Matrix/COL11 -> COL11
- MX72 pad 1: /Sheet: Switch Matrix/COL12 -> COL12
- MX73 pad 1: /Sheet: Switch Matrix/COL12 -> COL12
- MX74 pad 1: /Sheet: Switch Matrix/COL12 -> COL12
- MX75 pad 1: /Sheet: Switch Matrix/COL12 -> COL12
- MX76 pad 1: /Sheet: Switch Matrix/COL12 -> COL12
- MX77 pad 1: /Sheet: Switch Matrix/COL13 -> COL13
- MX78 pad 1: /Sheet: Switch Matrix/COL13 -> COL13
- MX79 pad 1: /Sheet: Switch Matrix/COL13 -> COL13
- MX8 pad 1: /Sheet: Switch Matrix/COL1 -> COL1
- MX9 pad 1: /Sheet: Switch Matrix/COL1 -> COL1
- R2 pad 1: /D+ -> D+
- R3 pad 1: /D- -> D-
- U1 pad 10: unconnected-(U1-PB2-Pad10) -> ROW2
- U1 pad 11: unconnected-(U1-PB3-Pad11) -> ROW3
- U1 pad 18: unconnected-(U1-PD0-Pad18) -> COL13
- U1 pad 19: unconnected-(U1-PD1-Pad19) -> COL12
- U1 pad 20: unconnected-(U1-PD2-Pad20) -> ROW4
- U1 pad 21: unconnected-(U1-PD3-Pad21) -> ROW5
- U1 pad 22: unconnected-(U1-PD5-Pad22) -> COL11
- U1 pad 25: unconnected-(U1-PD4-Pad25) -> COL3
- U1 pad 26: unconnected-(U1-PD6-Pad26) -> COL4
- U1 pad 27: unconnected-(U1-PD7-Pad27) -> COL5
- U1 pad 28: unconnected-(U1-PB4-Pad28) -> COL6
- U1 pad 29: unconnected-(U1-PB5-Pad29) -> COL7
- U1 pad 30: unconnected-(U1-PB6-Pad30) -> COL8
- U1 pad 31: unconnected-(U1-PC6-Pad31) -> COL9
- U1 pad 32: unconnected-(U1-PC7-Pad32) -> COL10
- U1 pad 38: unconnected-(U1-PF5-Pad38) -> COL0
- U1 pad 39: unconnected-(U1-PF4-Pad39) -> COL1
- U1 pad 40: unconnected-(U1-PF1-Pad40) -> COL2
- U1 pad 8: unconnected-(U1-PB0-Pad8) -> ROW0
- U1 pad 9: unconnected-(U1-PB1-Pad9) -> ROW1
- USB1 pad 3: /D- -> D+
- USB1 pad 4: /D+ -> D-
Routing:
- net COL9: track 0.00 -> 487.3 mm, vias 0 -> 4
- net COL5: track 0.00 -> 484.2 mm, vias 0 -> 6
- net COL7: track 0.00 -> 478.1 mm, vias 0 -> 4
- net COL6: track 0.00 -> 473.9 mm, vias 0 -> 4
- net COL8: track 0.00 -> 466.4 mm, vias 0 -> 4
- net COL4: track 0.00 -> 461.2 mm, vias 0 -> 6
- net COL3: track 0.00 -> 459.7 mm, vias 0 -> 6
- net COL10: track 0.00 -> 444.6 mm, vias 0 -> 2
- net COL0: track 0.00 -> 428.7 mm, vias 0 -> 4
- net COL1: track 0.00 -> 416.7 mm, vias 0 -> 4
- net ROW5: track 0.00 -> 411.5 mm, vias 0 -> 2
- net COL2: track 0.00 -> 405.0 mm, vias 0 -> 4
- net ROW4: track 0.00 -> 359.5 mm, vias 0 -> 2
- net ROW0: track 0.00 -> 333.2 mm, vias 0 -> 2
- net ROW3: track 0.00 -> 328.6 mm, vias 0 -> 2
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Other:
- board outline added: 314.3 x 114.4 mm
