File: Keyboard_v2/Keyboard_v2.kicad_pcb (KiCad board)
At the start: 2 copper layers, 162 parts, among them U1 ProMicro

Commit message: all keys routed
Parts:
- D1, D10, D11, D12, D13, D14, D15, D16, D17, D18, D19, D2, D20, D21, D22, D23, D24, D25, D26, D27, D28, D29, D3, D30, D31, D32, D33, D34, D35, D36, D37, D38, D39, D4, D40, D41, D42, D43, D44, D45, D46, D47, D48, D49, D5, D50, D51, D52, D53, D54, D55, D56, D57, D58, D59, D6, D60, D61, D62, D63, D64, D65, D66, D67, D68, D69, D7, D70, D71, D72, D73, D74, D75, D76, D77, D78, D79, D8, D9: moved to B.Cu
- moved S1 598.3 mm to (50.1, 158.1)
- moved MX70 576.9 mm to (57.3, 177.3)
- moved MX71 553.0 mm to (76.5, 177.3)
- moved MX69 552.4 mm to (38.2, 177.3)
- moved MX72 538.4 mm to (98.0, 177.3)
- moved MX56 530.4 mm to (50.1, 158.1)
- moved MX57 496.1 mm to (81.2, 158.1)
- moved MX58 474.0 mm to (100.4, 158.1)
- moved MX73 459.9 mm to (167.4, 177.2)
- moved MX59 452.6 mm to (119.5, 158.1)
- moved MX62 437.9 mm to (177.1, 158.1)
- moved D69 435.5 mm to (41.3, 177.8), turned to 90 degrees
- moved MX60 431.9 mm to (138.7, 158.1)
- moved D56 418.2 mm to (53.2, 158.8), turned to 90 degrees
- moved D43 417.8 mm to (48.4, 139.7), turned to 90 degrees
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Connections:
- MX74 pad 1: Net-(MX22-Pad1) -> Net-(MX23-Pad1)
- MX75 pad 1: Net-(MX23-Pad1) -> Net-(MX10-Pad1)
- MX76 pad 1: Net-(MX10-Pad1) -> Net-(MX11-Pad1)
- MX77 pad 1: Net-(MX11-Pad1) -> Net-(MX12-Pad1)
- MX78 pad 1: Net-(MX12-Pad1) -> Net-(MX13-Pad1)
- MX79 pad 1: Net-(MX13-Pad1) -> Net-(MX14-Pad1)
Routing:
- net Net-(D69-K): track 0.00 -> 310.1 mm
- net Net-(D56-K): track 0.00 -> 281.1 mm
- net Net-(D1-K): track 0.00 -> 270.8 mm
- net Net-(D15-K): track 0.00 -> 270.6 mm
- net Net-(D29-K): track 0.00 -> 270.5 mm
- net Net-(D43-K): track 0.00 -> 259.6 mm
- net Net-(MX19-Pad1): track 0.00 -> 133.1 mm
- net Net-(MX16-Pad1): track 0.00 -> 129.0 mm
- net Net-(MX13-Pad1): track 0.00 -> 127.8 mm
- net Net-(MX12-Pad1): track 0.00 -> 127.7 mm
- net Net-(MX10-Pad1): track 0.00 -> 126.9 mm
- net Net-(MX11-Pad1): track 0.00 -> 126.9 mm
- net Net-(MX23-Pad1): track 0.00 -> 126.4 mm
- net Net-(MX17-Pad1): track 0.00 -> 125.4 mm
- net Net-(MX18-Pad1): track 0.00 -> 124.0 mm
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