File: Keyboard_v2/_autosave-Keyboard_v2.kicad_pcb (KiCad board)
At the start: 2 copper layers, 316.2 x 114.9 mm, 177 parts, among them SW1 SW_Push, U1 ATmega32U4-A, Y1 16MHz

Commit message: pcb is routed and ground fills added
Parts:
- moved D10 0.31 mm to (223.3, 82.3)
Other:
- board size 316.2 x 114.9 mm -> 316.1 x 114.9 mm
